Commit message: new empty world launch and description package simplification

File: tello_description/urdf/tello.urdf (robot description, URDF)
Before this commit: robot tello${suffix}, 2 links, 1 joints
Links:
- removed link base_link${suffix}
- removed link camera_link${suffix}
- added link base_link, mass 0.1; collision box size=0.18 0.18 0.05; visual box size=0.07 0.02 0.02
- added link camera_link, mass 1e-5; collision sphere radius=0.01; visual sphere radius=0.01
Joints:
- removed joint camera_joint${suffix}
- added joint camera_joint: type fixed, parent base_link, child camera_link, origin xyz=0.035 0 0 rpy=0 0 0

Commit message: xacro added to the urdf and gitignore update

File: tello_description/urdf/tello.urdf (robot description, URDF)
Before this commit: robot tello, 2 links, 1 joints
Links:
- added link base_footprint
- added link dummy_link, mass 0.1
- link base_link: mass 0.1 -> None
Joints:
- added joint base_joint: type fixed, parent base_link, child base_footprint, origin xyz=0.0 0.0 0.0 rpy=0 0 0
- added joint dummy_joint: type fixed, parent base_link, child dummy_link
